Commit message: Confirmed: Commenting out Can link

File: bumperbot_description/urdf/bumperbot.urdf.xacro (robot description, xacro)
@@ -69,5 +69,5 @@
     <origin rpy = "0 0 0" xyz = "-0.04755 0 -0.0275"/>
 </joint>
-<link name = "can_link">
+<!-- <link name = "can_link">
     <visual>
         <origin rpy = "1.57 0 0" xyz = "-0.03 0.03 0"/>
@@ -81,4 +81,4 @@
     <child link = "can_link"/>
     <origin rpy = "0 0 0" xyz = "0 0 0.078"/>
-</joint>
+</joint> -->
 </robot>

Commit message: Added 5 mm to the can link

File: bumperbot_description/urdf/bumperbot.urdf.xacro (robot description, xacro)
@@ -71,5 +71,5 @@
 <!-- <link name = "can_link">
     <visual>
-        <origin rpy = "1.57 0 0" xyz = "-0.03 0.03 0"/>
+        <origin rpy = "1.57 0 0" xyz = "-0.035 0.035 0"/>
         <geometry>
             <mesh filename = "package://bumperbot_description/meshes/can.STL"/>

Commit message: Added the Gazebo launch file

File: bumperbot_description/urdf/bumperbot.urdf.xacro (robot description, xacro)
@@ -1,12 +1,26 @@
 <?xml version = "1.0"?>
 <robot xmlns:xacro = "http//www.ros.org/wiki/xacro" name = "bumperbot">
+<xacro:include filename = "$(find bumperbot_description)/urdf/bumperbot_gazebo.xacro"/>
 <link name = "base_footprint"/>
 <link name = "base_link">
-    <visual>
-        <origin rpy = "0 0 0" xyz = "0 0 0"/>
-        <geometry>
-            <mesh filename = "package://bumperbot_description/meshes/base_link.STL"/>
-        </geometry>
-    </visual>
+        <inertial>
+        <origin xyz="0 0 0.04" rpy="0.0 0.25 0.3" />
+        <mass value="8.2573504e-01"/>
+        <inertia ixx="2.2124416e-02" ixy="-1.2294101e-04" ixz="3.4938785e-04"
+                iyy="2.1193702e-02" iyz="-5.0120904e-05"
+                izz="2.0064271e-02" />
+        </inertial>
+        <visual>
+            <origin rpy = "0 0 0" xyz = "0 0 0"/>
+            <geometry>
+                <mesh filename = "package://bumperbot_description/meshes/base_link.STL"/>
+            </geometry>
+        </visual>
+        <collision>
+            <origin xyz = "0 0 0"  rpy = "0 0 0"/>
+            <geometry>
+                <mesh filename = "package://bumperbot_description/meshes/base_link.STL"/>
+            </geometry>
+        </collision>
 </link>
 <joint name = "base_joint" type = "fixed">
@@ -16,10 +30,23 @@
 </joint>
 <link name = "wheel_right_link">
-    <visual>
-        <origin rpy = "1.57 0 0" xyz = "0 0 0"/>
-        <geometry>
-            <mesh filename = "package://bumperbot_description/meshes/wheel_right_link.STL"/>
-        </geometry>
-    </visual>
+        <inertial>
+        <origin xyz="0 -0.014 0" rpy="0 0 0" />
+        <mass value="0.0530086090966721" />
+        <inertia ixx="1.88176298336665E-05" ixy="-4.8444933029987E-10" ixz="1.88163708851143E-08"
+                iyy="3.11510738647764E-05" iyz="-6.93560663069607E-11"
+                izz="1.8801969558182E-05" />
+        </inertial>
+        <visual>
+            <origin rpy = "1.57 0 0" xyz = "0 0 0"/>
+            <geometry>
+                <mesh filename = "package://bumperbot_description/meshes/wheel_right_link.STL"/>
+            </geometry>
+        </visual>
+        <collision>
+            <origin rpy = "1.57 0 0" xyz = "0 -0.015 0"/>
+            <geometry>
+                <sphere radius = "0.033"/>
+            </geometry>
+        </collision>
 </link>
 <joint name = "wheel_right_joint" type = "continuous">
@@ -30,10 +57,23 @@
 </joint>
 <link name = "wheel_left_link">
-    <visual>
-        <origin rpy = "-1.57 0 0" xyz = "0 0 0"/>
-        <geometry>
-            <mesh filename = "package://bumperbot_description/meshes/wheel_left_link.STL"/>
-        </geometry>
-    </visual>
+    <inertial>
+        <origin xyz="0 0.014 0" rpy="0 0 0" />
+        <mass value="0.0530086043217644" />
+        <inertia ixx="1.8792911368909E-05"  ixy="3.31256392204584E-10" ixz="-1.14082001662767E-08"
+                iyy="3.11510738759073E-05" iyz="-3.60499245082192E-10"
+                izz="1.88266886146847E-05" />
+        </inertial>
+        <visual>
+            <origin rpy = "-1.57 0 0" xyz = "0 0 0"/>
+            <geometry>
+                <mesh filename = "package://bumperbot_description/meshes/wheel_left_link.STL"/>
+            </geometry>
+        </visual>
+        <collision>
+            <origin rpy = "1.57 0 0" xyz = "0 00.015 0"/>
+            <geometry>
+                <sphere radius = "0.033"/>
+            </geometry>
+        </collision>
 </link>
 <joint name = "wheel_left_joint" type = "continuous">
@@ -44,10 +84,23 @@
 </joint>
 <link name = "caster_front_link">
-    <visual>
-        <origin rpy = "0 0 0" xyz = "0 0 0"/>
-        <geometry>
-            <mesh filename = "package://bumperbot_description/meshes/caster_front_link.STL"/>
-        </geometry>
-    </visual>
+        <inertial>
+        <origin xyz="3.89968128948481E-07 2.40073004698083E-07 0.00219173397061506" rpy="0 0 0" />
+        <mass value="1.44379265037903E-06" />
+        <inertia ixx="7.23075276010246E-11" ixy="-6.10956883467859E-16" ixz="2.22849693525031E-15"
+                iyy="3.8713793085917E-11"  iyz="2.93909858781952E-15"
+                izz="1.00967486676306E-10" />
+        </inertial>
+        <visual>
+            <origin rpy = "0 0 0" xyz = "0 0 0"/>
+            <geometry>
+                <mesh filename = "package://bumperbot_description/meshes/caster_front_link.STL"/>
+            </geometry>
+        </visual>
+        <collision>
+            <origin rpy = "0 0 0" xyz = "0 0 0"/>
+            <geometry>
+                <sphere radius = "0.005"/>
+            </geometry>
+        </collision>
 </link>
 <joint name = "caster_front_joint" type = "fixed">
@@ -57,10 +110,23 @@
 </joint>
 <link name = "caster_rear_link">
-    <visual>
-        <origin rpy = "0 0 0" xyz = "0 0 0"/>
-        <geometry>
-            <mesh filename = "package://bumperbot_description/meshes/caster_rear_link.STL"/>
-        </geometry>
-    </visual>
+        <inertial>
+        <origin xyz="3.8996812895542E-07 2.40073004698083E-07 0.00219173397061509" rpy="0 0 0" />
+        <mass value="1.44379265037902E-06" />
+        <inertia ixx="7.23075276010246E-11" ixy="-6.10956872363424E-16" ixz="2.22849693527207E-15"
+                iyy="3.87137930859167E-11" iyz="2.939098587861E-15"
+                izz="1.00967486676306E-10" />
+        </inertial>
+        <visual>
+            <origin rpy = "0 0 0" xyz = "0 0 0"/>
+            <geometry>
+                <mesh filename = "package://bumperbot_description/meshes/caster_rear_link.STL"/>
+            </geometry>
+        </visual>
+        <collision>
+            <origin rpy = "0 0 0" xyz = "0 0 0"/>
+            <geometry>
+                <sphere radius = "0.005"/>
+            </geometry>
+        </collision>
 </link>
 <joint name = "caster_rear_joint" type = "fixed">
@@ -69,16 +135,3 @@
     <origin rpy = "0 0 0" xyz = "-0.04755 0 -0.0275"/>
 </joint>
-<!-- <link name = "can_link">
-    <visual>
-        <origin rpy = "1.57 0 0" xyz = "-0.035 0.035 0"/>
-        <geometry>
-            <mesh filename = "package://bumperbot_description/meshes/can.STL"/>
-        </geometry>
-    </visual>
-</link>
-<joint name = "can_joint" type = "fixed">
-    <parent link = "base_link"/>
-    <child link = "can_link"/>
-    <origin rpy = "0 0 0" xyz = "0 0 0.078"/>
-</joint> -->
 </robot>

Commit message: Added the .yaml file for the controller manager and linked it with the bumperbot_gazebo.xacro file

File: bumperbot_description/urdf/bumperbot.urdf.xacro (robot description, xacro)
@@ -1,5 +1,9 @@
 <?xml version = "1.0"?>
 <robot xmlns:xacro = "http//www.ros.org/wiki/xacro" name = "bumperbot">
+<xacro:arg name = "is_ignition" default = "true"/>
+<!--Include Gazebo Parameters-->
 <xacro:include filename = "$(find bumperbot_description)/urdf/bumperbot_gazebo.xacro"/>
+<!--Include ROS2 Control Plugins-->
+<xacro:include filename = "$(find bumperbot_description)/urdf/bumperbot_ros2_control.xacro"/>
 <link name = "base_footprint"/>
 <link name = "base_link">

File: bumperbot_description/urdf/bumperbot_gazebo.xacro (robot description, xacro)
@@ -40,10 +40,10 @@
    <xacro:if value = "$(arg is_ignition)">
       <plugin filename = "ign_ros2_control-system" name = "ign_ros2_control::IgnitionROS2ControlPlugin">
-         <parameters></parameters>
+         <parameters>$(find bumperbot_controller)/config/bumperbot_controllers.yaml</parameters>
       </plugin>
    </xacro:if>
    <xacro:unless value = "$(arg is_ignition)">
       <plugin filename = "gz_ros2_control-system" name = "gz_ros2_control::GazeboSimROS2ControlPlugin">
-         <parameters></parameters>
+         <parameters>$(find bumperbot_controller)/config/bumperbot_controllers.yaml</parameters>
       </plugin>
    </xacro:unless>

File: bumperbot_description/urdf/bumperbot_ros2_control.xacro (robot description, xacro)
@@ -1,5 +1,5 @@
 <?xml version = "1.0" ?>
 <robot xmlns:xacro = "http://www.ros.org/wiki/xacro" name = "bumperbot">
-<ros2_control>
+<ros2_control name = "RobotSystem" type = "system">
     <xacro:if value = "$(arg is_ignition)">
         <hardware>
@@ -12,20 +12,20 @@
         </hardware>
     </xacro:unless>
+    <joint name = "wheel_right_joint">
+        <command_interface name = "velocity">
+            <param name = "min">-1</param>
+            <param name = "max">1</param>
+        </command_interface>
+        <state_interface name = "position"/>
+        <state_interface name = "velocity"/>
+    </joint>
+    <joint name = "wheel_left_joint">
+        <command_interface name = "velocity">
+            <param name = "min">-1</param>
+            <param name = "max">1</param>
+        </command_interface>
+        <state_interface name = "position"/>
+        <state_interface name = "velocity"/>
+    </joint>
 </ros2_control>
-<joint name = "wheel_right_joint">
-    <command_interface name = "velocity">
-        <param name = "min">-1</param>
-        <param name = "max">1</param>
-    </command_interface>
-    <state_interface name = "position"/>
-    <state_interface name = "velocity"/>
-</joint>
-<joint name = "wheel_left_joint">
-    <command_interface name = "velocity">
-        <param name = "min">-1</param>
-        <param name = "max">1</param>
-    </command_interface>
-    <state_interface name = "position"/>
-    <state_interface name = "velocity"/>
-</joint>
 </robot>
